File: gpio_isolated_switches.kicad_pcb (KiCad board)
At the start: 2 copper layers, 29.4 x 52 mm, 38 parts, among them J1 Conn_01x02, J2 Conn_01x02, J3 Conn_01x02, J4 Conn_01x02, J5 SBC GPIO, J6 Conn_01x02, Q1 BUK7M10-40EX, Q2 BUK7M10-40EX, Q3 BUK7M10-40EX, Q4 BUK7M10-40EX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

Commit message: Adding SW0 direct output from optocoupler
Parts:
- added J7: Conn_01x02, Connector_PinHeader_2.54mm:PinHeader_1x02_P2.54mm_Vertical, F.Cu at (97.0, 76.5)
- added R12: 0R, Resistor_SMD:R_0603_1608Metric, B.Cu at (94.2, 76.2)
- moved R5 3.33 mm to (92.8, 83.7)
- moved C1 2.45 mm to (93.5, 78.7)
- moved Q1 2.45 mm to (97.0, 80.6)
- moved U2 2.45 mm to (93.0, 81.2)
- moved U1 0.60 mm to (94.5, 69.2)
Connections:
- U1 pad 16: +12V -> Net-(U1-Pad16)
Routing:
- net Net-(U1-Pad16): track 0.00 -> 6.52 mm
- net Net-(J1-Pad2): track 9.02 -> 10.0 mm
- net Net-(R5-Pad1): track 17.9 -> 18.9 mm, vias 2 -> 1
- net Net-(R8-Pad1): track 26.0 -> 25.4 mm
