File: gpio_isolated_switches.kicad_pcb (KiCad board)
At the start: 2 copper layers, 29.4 x 52 mm, 40 parts, among them J1 Conn_01x02, J2 Conn_01x02, J3 Conn_01x02, J4 Conn_01x02, J5 SBC GPIO, J6 Conn_01x02, J7 Conn_01x02, Q1 BUK7M10-40EX, Q2 BUK7M10-40EX, Q3 BUK7M10-40EX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

Commit message: Removed SW0 switch, left direct optocoupler output only
Parts:
- removed C1: 100n 25V, Capacitor_SMD:C_0603_1608Metric
- removed J1: Conn_01x02, TerminalBlock:TerminalBlock_Altech_AK300-2_P5.00mm
- removed Q1: BUK7M10-40EX, Package_TO_SOT_SMD:LFPAK33
- removed R12: 0R, Resistor_SMD:R_0603_1608Metric
- removed R5: 10k, Resistor_SMD:R_0603_1608Metric
- removed U2: MCP1416, Package_TO_SOT_SMD:SOT-23-5
- J7: footprint Connector_PinHeader_2.54mm:PinHeader_1x02_P2.54mm_Vertical -> Connector_PinHeader_2.54mm:PinHeader_1x02_P2.54mm_Horizontal
- moved J7 2.17 mm to (98.8, 77.8), turned to 0 degrees
Connections:
- J7 pad 1: Net-(U1-Pad16) -> Net-(J7-Pad1)
- J7 pad 2: Net-(R5-Pad1) -> Net-(J7-Pad2)
- U1 pad 15: Net-(R5-Pad1) -> Net-(J7-Pad1)
- U1 pad 16: Net-(U1-Pad16) -> Net-(J7-Pad2)
Routing:
- net +12V: track 91.2 -> 70.7 mm, vias 6 -> 0
- net Net-(R5-Pad1): track 18.9 -> 0.00 mm, vias 1 -> 0
- net Net-(J1-Pad2): track 10.0 -> 0.00 mm
- net Net-(J7-Pad2): track 0.00 -> 7.22 mm
- net Net-(U1-Pad16): track 6.52 -> 0.00 mm
- net Net-(J7-Pad1): track 0.00 -> 6.47 mm
- net Net-(Q1-Pad4): track 1.89 -> 0.00 mm

Commit message: Adding DS18B20 as an optional temperature sensor
Parts:
- added R5: 10k, Resistor_SMD:R_0603_1608Metric, F.Cu at (90.8, 60.3)
- added U2: DS18S20, Package_TO_SOT_THT:TO-92_Inline, F.Cu at (89.5, 55.2)
Connections:
- J5 pad 15: unconnected-(J5-Pad15) -> /OneWire
- J5 pad 6: unconnected-(J5-Pad6) -> GND
Routing:
- net /OneWire: track 0.00 -> 16.3 mm
- net +3V3: track 19.7 -> 32.9 mm
- net GND: track 27.7 -> 35.2 mm
Other:
- board text added: "Isolated 24V low side switches Also temperature sensor for Odroid M1 Tomek Szczęsny 2022"
- board text removed: "Isolated 24V low side switches Also temperature sensors because why not for Odroids Tomek Szczęsny 2022"
